File: pressure_strips/pressure_strips.kicad_pcb (KiCad board)
At the start: 4 copper layers, 357.3 x 17.2 mm, 41 parts, among them J1 Conn_01x05, U1 ILPS28QSW, U2 ILPS28QSW, U3 ILPS28QSW, U4 ILPS28QSW, U5 ILPS28QSW, U6 ILPS28QSW, U7 TCA9548APWR, U9 ILPS28QSW

Commit message: initial commit
Other:
- board text added: "User drawn rectangles under sensors stiffened with FR4"

Commit message: strips done, finishing off mcu
Parts:
- J1: footprint Connector_JST:JST_EH_B5B-EH-A_1x05_P2.50mm_Vertical -> Connector_PinHeader_2.00mm:PinHeader_1x05_P2.00mm_Vertical_SMD_Pin1Left
- moved J1 5.51 mm to (31.4, 142.6), turned to 180 degrees
Routing:
- net +3V3: track 23.0 -> 27.2 mm
- net /MUX_SDA: track 5.11 -> 6.64 mm
- net /MUX_NRST: track 8.53 -> 9.89 mm
- net /MUX_SCL: track 4.50 -> 3.30 mm
Other:
- board text added: "J. Tomkins"
