File: pressure_strips/pressure_strips.kicad_sch (KiCad schematic)
At the start: 46 parts, among them J1 Conn_01x05, U1 ILPS28QSW, U2 ILPS28QSW, U3 ILPS28QSW, U4 ILPS28QSW, U5 ILPS28QSW, U6 ILPS28QSW, U7 TCA9548APWR, U8 ILPS28QSW, U9 ILPS28QSW

Commit message: strips done, finishing off mcu
Parts:
- J1: footprint Connector_JST:JST_EH_B5B-EH-A_1x05_P2.50mm_Vertical -> Connector_PinHeader_2.00mm:PinHeader_1x05_P2.00mm_Vertical_SMD_Pin1Left
Other:
- note added: "Connector"
- note added: "I2C Switch"
- note added: "Wires will be soldered down and stiffened with epoxy"
- moved on the sheet: C1, C10, C11, C12, C13, C14, C15, C16, C17, C18, C2, C3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
