File: pressure_mcu/pressure_mcu.kicad_pcb (KiCad board)
At the start: 2 copper layers, 33.2 x 35 mm, 23 parts, among them J1 USB_C_Receptacle_USB2.0_14P, J4 Connector 1, J5 Connector 2, J6 Connector 3, J7 Connector 4, U1 STM32H563RITx, U2 AP2112K-3.3

Commit message: strips done, finishing off mcu
Parts:
- removed C1, C10, C11, C12, C2, C3, C4, C5, C6, C7, C8, C9: C, Capacitor_SMD:C_0402_1005Metric
- removed U1: STM32H563RITx, Package_QFP:LQFP-64_10x10mm_P0.5mm
- added C23: 100nF, Capacitor_SMD:C_0603_1608Metric, F.Cu at (177.5, 91.1)
- added C24: 4.7uF, Capacitor_SMD:C_0603_1608Metric, F.Cu at (182.1, 86.2)
- added C25: 100nF, Capacitor_SMD:C_0603_1608Metric, F.Cu at (192.9, 89.6)
- added C26: 4.7uF, Capacitor_SMD:C_0603_1608Metric, F.Cu at (191.8, 100.6)
- added C27: 100nF, Capacitor_SMD:C_0603_1608Metric, F.Cu at (179.3, 99.5)
- added C28: 4.7uF, Capacitor_SMD:C_0603_1608Metric, F.Cu at (177.5, 92.7)
- added C29: 100nF, Capacitor_SMD:C_0603_1608Metric, F.Cu at (183.6, 85.7)
- added C30: 4.7uF, Capacitor_SMD:C_0603_1608Metric, F.Cu at (191.8, 88.0)
- added C31: 27pF, Capacitor_SMD:C_0603_1608Metric, F.Cu at (191.1, 85.7)
- added C32: 27pF, Capacitor_SMD:C_0603_1608Metric, F.Cu at (185.2, 86.2)
- added C33: 2u2, Resistor_SMD:R_0603_1608Metric, F.Cu at (177.8, 97.3)
- added C34: 2u2, Resistor_SMD:R_0603_1608Metric, F.Cu at (194.4, 91.2)
- added D2: LED_R, LED_SMD:LED_0603_1608Metric, F.Cu at (177.6, 111.0)
- added D3: LED_G, LED_SMD:LED_0603_1608Metric, F.Cu at (179.1, 111.0)
- added J8: SWD JST PH, Connector_JST:JST_PH_B4B-PH-K_1x04_P2.00mm_Vertical, F.Cu at (200.3, 102.4)
- added R12: 10k, Resistor_SMD:R_0603_1608Metric, F.Cu at (194.4, 92.8)
- added R15: 220R, Resistor_SMD:R_0603_1608Metric, F.Cu at (179.1, 107.9)
- added R16: 220R, Resistor_SMD:R_0603_1608Metric, F.Cu at (177.6, 107.9)
- added U4: STM32H562RGT6, Package_QFP:LQFP-64_10x10mm_P0.5mm, F.Cu at (186.1, 94.5)
- added Y2: 12MHz, Crystal:Crystal_SMD_Abracon_ABM8G-4Pin_3.2x2.5mm, F.Cu at (188.1, 85.9)
- moved R2 7.10 mm to (192.2, 109.6)
- moved R4 2.77 mm to (184.8, 103.8), turned to 0 degrees
- moved R3 0.83 mm to (184.3, 105.4)
Connections:
- net Net-(U2-EN) renamed /V_BUS
- J1 pad A6: /USB_D+ -> unconnected-(J1-D+-PadA6)
- J1 pad A7: /USB_D- -> unconnected-(J1-D--PadA7)
- J1 pad B6: unconnected-(J1-D+-PadB6) -> /USB_D+
- J1 pad B7: unconnected-(J1-D--PadB7) -> /USB_D-
Routing:
- net GND: track 0.00 -> 29.3 mm, vias 0 -> 24
- net +3V3: track 0.00 -> 22.7 mm, vias 0 -> 7
- net /V_BUS: track 0.00 -> 11.6 mm
- net Net-(U4-PH0): track 0.00 -> 6.42 mm
- net Net-(J1-CC2): track 0.00 -> 5.62 mm
- net /USB_D+: track 0.00 -> 4.63 mm
- net Net-(U4-PH1): track 0.00 -> 4.13 mm
- net /USB_D-: track 0.00 -> 4.13 mm, vias 0 -> 2
- net Net-(J1-CC1): track 0.00 -> 2.19 mm
- net Net-(C34-Pad1): track 0.00 -> 2.03 mm
- net Net-(C33-Pad1): track 0.00 -> 1.83 mm
- net Net-(U4-BOOT0): track 0.00 -> 1.80 mm
- net Net-(D3-A): track 0.00 -> 1.47 mm
- net Net-(D2-A): track 0.00 -> 1.47 mm
- net /V_SENSE: track 0.00 -> 1.04 mm
- added copper zone on B.Cu, net +3V3
- added copper zone on F.Cu, net GND

Commit message: pressure mcu schematic almost done
Parts:
- removed J1: USB_C_Receptacle_USB2.0_14P, Connector_USB:USB_C_Receptacle_Amphenol_124019772112A
- removed R1, R2: 5.1k, Resistor_SMD:R_0402_1005Metric
- added C17: 4u7F, Capacitor_SMD:C_0402_1005Metric, F.Cu at (191.8, 86.6)
- added C18: 100nF, Capacitor_SMD:C_0402_1005Metric, F.Cu at (191.8, 84.7)
- added J2: USB_B_Micro, Connector_USB:USB_Micro-B_Amphenol_10118193-0001LF_Horizontal, F.Cu at (185.2, 111.5)
- added R10: R, Resistor_SMD:R_0402_1005Metric, F.Cu at (176.0, 84.4)
- added R11: R, Resistor_SMD:R_0402_1005Metric, B.Cu at (175.9, 92.6)
- added R13: R, Resistor_SMD:R_0402_1005Metric, B.Cu at (175.9, 93.6)
- added R17: 2.2k, Resistor_SMD:R_0402_1005Metric, F.Cu at (194.0, 99.6)
- added R18: 2.2k, Resistor_SMD:R_0402_1005Metric, F.Cu at (194.0, 98.6)
- added R5: R, Resistor_SMD:R_0402_1005Metric, B.Cu at (196.6, 90.4)
- added R6: R, Resistor_SMD:R_0402_1005Metric, F.Cu at (196.9, 83.4)
- added R7: R, Resistor_SMD:R_0402_1005Metric, F.Cu at (196.9, 82.4)
- added R8: R, Resistor_SMD:R_0402_1005Metric, B.Cu at (196.6, 91.5)
- added R9: R, Resistor_SMD:R_0402_1005Metric, F.Cu at (176.0, 83.4)
- added U7: TCA9548APWR, Package_SO:TSSOP-24_4.4x7.8mm_P0.65mm, F.Cu at (187.1, 83.7)
- J4: value Connector 1 -> 1; footprint Connector_JST:JST_EH_B5B-EH-A_1x05_P2.50mm_Vertical -> Connector_Wuerth:Wuerth_WR-WTB_64800511622_1x05_P1.50mm_Vertical
- J5: value Connector 2 -> 2; footprint Connector_JST:JST_EH_B5B-EH-A_1x05_P2.50mm_Vertical -> Connector_Wuerth:Wuerth_WR-WTB_64800511622_1x05_P1.50mm_Vertical
- J6: value Connector 3 -> 3; footprint Connector_JST:JST_EH_B5B-EH-A_1x05_P2.50mm_Vertical -> Connector_Wuerth:Wuerth_WR-WTB_64800511622_1x05_P1.50mm_Vertical
- J7: value Connector 4 -> 4; footprint Connector_JST:JST_EH_B5B-EH-A_1x05_P2.50mm_Vertical -> Connector_Wuerth:Wuerth_WR-WTB_64800511622_1x05_P1.50mm_Vertical
- J8: footprint Connector_JST:JST_PH_B4B-PH-K_1x04_P2.00mm_Vertical -> Connector:Tag-Connect_TC2050-IDC-NL_2x05_P1.27mm_Vertical_with_bottom_clip
- moved J6 16.2 mm to (173.0, 80.4), turned to -90 degrees
- moved D2 13.9 mm to (191.5, 111.0)
- moved D3 13.9 mm to (193.0, 111.0)
- moved R15 13.9 mm to (193.1, 107.9)
- moved R16 13.9 mm to (191.5, 107.9)
- moved U2 11.9 mm to (178.8, 109.9), turned to -90 degrees
- moved J5 11.9 mm to (199.7, 86.5), turned to 90 degrees
- moved J7 10.1 mm to (173.0, 90.6), turned to -90 degrees
- moved R3 6.65 mm to (177.8, 106.8)
- moved R4 6.65 mm to (178.8, 106.8), turned to -90 degrees
- moved C25 4.45 mm to (192.7, 94.0)
- moved C26 4.45 mm to (191.6, 105.0)
- moved C30 4.45 mm to (191.6, 92.4)
- moved C34 4.45 mm to (194.2, 95.7)
- moved U4 4.45 mm to (185.9, 99.0)
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Connections:
- J4 pad 2: /MUX1_NRST -> /MUX2_NRST
- J4 pad 3: /MUX1_SCL -> /MUX2_SCL
- J4 pad 4: /MUX1_SDA -> /MUX2_SDA
- J5 pad 2: /MUX2_NRST -> /MUX1_NRST
- J5 pad 3: /MUX2_SCL -> /MUX1_SCL
- J5 pad 4: /MUX2_SDA -> /MUX1_SDA
- U4 pad 58: unconnected-(U4-PB6-Pad58) -> /MUX_SCL
- U4 pad 59: unconnected-(U4-PB7-Pad59) -> /MUX_SDA
Routing:
- net /NRST: track 0.00 -> 21.4 mm, vias 0 -> 2
- net Net-(U7-SD3): track 0.00 -> 16.6 mm, vias 0 -> 1
- net Net-(U7-SCL): track 0.00 -> 16.4 mm, vias 0 -> 2
- net Net-(U7-SDA): track 0.00 -> 15.0 mm, vias 0 -> 2
- net Net-(U7-SC3): track 0.00 -> 15.0 mm, vias 0 -> 1
- net Net-(U7-SC0): track 0.00 -> 14.4 mm, vias 0 -> 1
- net Net-(U7-SD0): track 0.00 -> 13.3 mm, vias 0 -> 1
- net Net-(U7-SD2): track 0.00 -> 11.8 mm
- net /SWDIO: track 0.00 -> 11.7 mm
- net Net-(U7-SC1): track 0.00 -> 11.6 mm
- net Net-(U7-SD1): track 0.00 -> 11.5 mm
- net Net-(U7-SC2): track 0.00 -> 11.5 mm
- net /SWCLK: track 0.00 -> 8.02 mm
- net Net-(J1-CC2): track 5.62 -> 0.00 mm
- net +3V3: track 22.7 -> 26.3 mm, vias 7 -> 8
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
Commit message: ready for review
Parts:
- removed J6: 3, Connector_Wuerth:Wuerth_WR-WTB_64800511622_1x05_P1.50mm_Vertical
- removed J8: SWD JST PH, Connector:Tag-Connect_TC2050-IDC-NL_2x05_P1.27mm_Vertical_with_bottom_clip
- removed U4: STM32H562RGT6, Package_QFP:LQFP-64_10x10mm_P0.5mm
- removed U7: TCA9548APWR, Package_SO:TSSOP-24_4.4x7.8mm_P0.65mm
- added C35: 10uF, Capacitor_SMD:C_0603_1608Metric, F.Cu at (147.2, 118.2)
- added C36: 100nF, Capacitor_SMD:C_0402_1005Metric, F.Cu at (127.5, 114.7)
- added H1: MountingHole, MountingHole:MountingHole_2.2mm_M2, F.Cu at (122.6, 77.6)
- added H2: MountingHole, MountingHole:MountingHole_2.2mm_M2, F.Cu at (177.4, 77.6)
- added H3: MountingHole, MountingHole:MountingHole_2.2mm_M2, F.Cu at (122.6, 122.4)
- added H4: MountingHole, MountingHole:MountingHole_2.2mm_M2, F.Cu at (177.4, 122.4)
- added J1: 1, Connector_JST:JST_GH_SM05B-GHS-TB_1x05-1MP_P1.25mm_Horizontal, F.Cu at (167.1, 78.4)
- added J3: 3, Connector_JST:JST_GH_SM05B-GHS-TB_1x05-1MP_P1.25mm_Horizontal, F.Cu at (143.9, 78.4)
- added JP1: SolderJumper_2_Open, Jumper:SolderJumper-2_P1.3mm_Open_RoundedPad1.0x1.5mm, F.Cu at (176.8, 94.0)
- added JP2: SolderJumper_2_Open, Jumper:SolderJumper-2_P1.3mm_Open_RoundedPad1.0x1.5mm, F.Cu at (176.8, 91.5)
- added JP3: SolderJumper_2_Open, Jumper:SolderJumper-2_P1.3mm_Open_RoundedPad1.0x1.5mm, F.Cu at (176.8, 88.8)
- added R1: 10k, Resistor_SMD:R_0402_1005Metric, F.Cu at (130.1, 82.6)
- added R14: 0, Resistor_SMD:R_0402_1005Metric, F.Cu at (156.6, 82.7)
- added R19: 0, Resistor_SMD:R_0402_1005Metric, F.Cu at (168.2, 82.7)
- added R2: 2.2k, Resistor_SMD:R_0402_1005Metric, F.Cu at (131.2, 82.6)
- added R20: 2.2k, Resistor_SMD:R_0402_1005Metric, F.Cu at (169.2, 82.7)
- added R21: 10k, Resistor_SMD:R_0402_1005Metric, F.Cu at (144.2, 120.5)
- added R22: 15k, Resistor_SMD:R_0402_1005Metric, F.Cu at (142.2, 120.5)
- added R23: 220R, Resistor_SMD:R_0603_1608Metric, F.Cu at (160.4, 119.9)
- added R24: 220R, Resistor_SMD:R_0603_1608Metric, F.Cu at (162.0, 119.9)
- added R25: 10k, Resistor_SMD:R_0603_1608Metric, F.Cu at (154.4, 97.0)
- added R26: 2.2k, Resistor_SMD:R_0402_1005Metric, F.Cu at (155.6, 98.7)
- added R27: 2.2k, Resistor_SMD:R_0402_1005Metric, F.Cu at (156.5, 96.8)
- added R29: 10k, Resistor_SMD:R_0402_1005Metric, F.Cu at (171.9, 89.2)
- added R30: 10k, Resistor_SMD:R_0402_1005Metric, F.Cu at (174.6, 89.2)
- added R31: 10k, Resistor_SMD:R_0402_1005Metric, F.Cu at (174.6, 91.8)
- added R32: 10k, Resistor_SMD:R_0402_1005Metric, F.Cu at (174.6, 93.8)
- added U1: STM32H562RGT6, Package_QFP:LQFP-64_10x10mm_P0.5mm, F.Cu at (150.0, 105.0)
- added U3: AP2112K-3.3, Package_TO_SOT_SMD:SOT-23-5, F.Cu at (143.1, 122.8)
- C17: value 4u7F -> 4.7uF
- C31, C32: value 27pF -> 33pF
- C33, C34: value 2u2 -> 2.2uF; footprint Resistor_SMD:R_0603_1608Metric -> Capacitor_SMD:C_0603_1608Metric
- J2: value USB_B_Micro -> 2; footprint Connector_USB:USB_Micro-B_Amphenol_10118193-0001LF_Horizontal -> Connector_JST:JST_GH_SM05B-GHS-TB_1x05-1MP_P1.25mm_Horizontal
- J4: value 1 -> 4; footprint Connector_Wuerth:Wuerth_WR-WTB_64800511622_1x05_P1.50mm_Vertical -> Connector_JST:JST_GH_SM05B-GHS-TB_1x05-1MP_P1.25mm_Horizontal
- J5: value 2 -> USB_B_Micro; footprint Connector_Wuerth:Wuerth_WR-WTB_64800511622_1x05_P1.50mm_Vertical -> Connector_USB:USB_Micro-B_Amphenol_10118193-0001LF_Horizontal
- J7: value 4 -> SWD JST PH; footprint Connector_Wuerth:Wuerth_WR-WTB_64800511622_1x05_P1.50mm_Vertical -> Connector:Tag-Connect_TC2050-IDC-NL_2x05_P1.27mm_Vertical_with_bottom_clip
- R10, R7: value R -> 2.2k
- R11: value R -> 10k; moved to F.Cu
- R12: value 10k -> 2.2k; footprint Resistor_SMD:R_0603_1608Metric -> Resistor_SMD:R_0402_1005Metric
- R13, R8: value R -> 0; moved to F.Cu
- R15: value 220R -> 2.2k; footprint Resistor_SMD:R_0603_1608Metric -> Resistor_SMD:R_0402_1005Metric
- R16: value 220R -> 10k; footprint Resistor_SMD:R_0603_1608Metric -> Resistor_SMD:R_0402_1005Metric
- R18: value 2.2k -> 0
- R3: value 10k -> 0
- R4: value 15k -> 0
- R5: value R -> 2.2k; moved to F.Cu
- R6: value R -> 10k
- R9: value R -> 0
- U2: value AP2112K-3.3 -> TCA9548APWR; footprint Package_TO_SOT_SMD:SOT-23-5 -> Package_SO:TSSOP-24_4.4x7.8mm_P0.65mm
- moved J4 69.9 mm to (132.2, 78.3), turned to 180 degrees
- moved R5 62.7 mm to (134.4, 82.6), turned to 90 degrees
- moved J5 62.0 mm to (150.0, 123.5), turned to 0 degrees
- moved R6 55.1 mm to (141.8, 82.6), turned to 90 degrees
- moved R7 54.0 mm to (142.9, 82.6), turned to 90 degrees
- moved R8 53.4 mm to (143.9, 82.6), turned to 90 degrees
- moved J7 53.2 mm to (124.1, 111.5), turned to 90 degrees
- moved C25 52.6 mm to (142.4, 109.1), turned to -135 degrees
- moved R3 51.6 mm to (132.2, 82.6)
- moved R4 51.6 mm to (133.3, 82.6), turned to 90 degrees
- moved C26 48.4 mm to (143.5, 110.3), turned to -135 degrees
- moved C31 45.0 mm to (146.4, 96.5), turned to -45 degrees
- moved Y2 44.5 mm to (144.1, 97.9), turned to -45 degrees
- moved J2 44.5 mm to (155.5, 78.4), turned to 180 degrees
- moved C32 44.1 mm to (141.8, 99.3), turned to 135 degrees
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Connections:
- J2 pad 1: /V_BUS -> GND
- J2 pad 2: /USB_D- -> /MUX1_SDA
- J2 pad 3: /USB_D+ -> /MUX1_SCL
- J2 pad 4: unconnected-(J2-ID-Pad4) -> /MUX1_NRST
- J2 pad 5: GND -> +3V3
- J4 pad 1: +3V3 -> GND
- J4 pad 2: /MUX2_NRST -> /MUX4_SDA
- J4 pad 3: /MUX2_SCL -> /MUX4_SCL
- J4 pad 4: /MUX2_SDA -> /MUX4_NRST
- J4 pad 5: GND -> +3V3
- J5 pad 1: +3V3 -> /V_BUS
- J5 pad 2: /MUX1_NRST -> /USB_D-
- J5 pad 3: /MUX1_SCL -> /USB_D+
- J5 pad 4: /MUX1_SDA -> unconnected-(J5-ID-Pad4)
- J7 pad 2: /MUX4_NRST -> /SWDIO
- J7 pad 3: /MUX4_SCL -> GND
- J7 pad 4: /MUX4_SDA -> /SWCLK
- R10 pad 1: Net-(U7-SD2) -> +3V3
- R11 pad 1: Net-(U7-SC3) -> +3V3
- R11 pad 2: /MUX4_SCL -> /MUX1_NRST
- R12 pad 1: Net-(U4-BOOT0) -> +3V3
- R12 pad 2: GND -> /MUX1_SCL
- R13 pad 1: Net-(U7-SD3) -> Net-(U2-SC1)
- R13 pad 2: /MUX4_SDA -> /MUX1_SCL
- R15 pad 1: /LED1 -> +3V3
- R15 pad 2: Net-(D3-A) -> /MUX1_SDA
- R16 pad 1: /LED2 -> +3V3
- R16 pad 2: Net-(D2-A) -> /MUX2_NRST
- R17 pad 1: Net-(U7-SCL) -> +3V3
- R17 pad 2: /MUX_SCL -> /MUX2_SCL
- R18 pad 1: Net-(U7-SDA) -> Net-(U2-SC0)
- R18 pad 2: /MUX_SDA -> /MUX2_SCL
- R3 pad 1: /V_BUS -> Net-(U2-SC3)
- R3 pad 2: /V_SENSE -> /MUX4_SCL
- R4 pad 1: /V_SENSE -> Net-(U2-SD3)
- R4 pad 2: GND -> /MUX4_SDA
- R5 pad 1: Net-(U7-SD0) -> +3V3
- R5 pad 2: /MUX2_SDA -> /MUX4_SDA
- R6 pad 1: Net-(U7-SC1) -> +3V3
- R6 pad 2: /MUX1_SCL -> /MUX3_NRST
- R7 pad 1: Net-(U7-SD1) -> +3V3
- R7 pad 2: /MUX1_SDA -> /MUX3_SCL
- R8 pad 1: Net-(U7-SC0) -> Net-(U2-SC2)
- R8 pad 2: /MUX2_SCL -> /MUX3_SCL
- R9 pad 1: Net-(U7-SC2) -> Net-(U2-SD2)
- R9 pad 2: /MUX3_SCL -> /MUX3_SDA
- U2 pad 1: /V_BUS -> /A0
- U2 pad 2: GND -> /A1
- U2 pad 3: /V_BUS -> /MUX_NRST
- U2 pad 4: unconnected-(U2-NC-Pad4) -> Net-(U2-SD0)
- U2 pad 5: +3V3 -> Net-(U2-SC0)
Routing:
- net Net-(U2-SC3): track 0.00 -> 38.1 mm
- net Net-(U2-SD3): track 0.00 -> 37.8 mm
- net /nRESET: track 0.00 -> 36.7 mm, vias 0 -> 2
- net /SWO: track 0.00 -> 35.0 mm
- net /V_SENSE: track 1.02 -> 35.3 mm, vias 0 -> 2
- net Net-(U2-SC2): track 0.00 -> 27.9 mm
- net Net-(U2-SD2): track 0.00 -> 27.7 mm
- net /SWCLK: track 8.02 -> 34.6 mm
- net /SWDIO: track 11.7 -> 34.2 mm, vias 0 -> 2
- net /LED2: track 0.00 -> 22.1 mm
- net /NRST: track 21.4 -> 0.00 mm, vias 2 -> 0
- net /LED1: track 0.00 -> 21.4 mm
- net /MUX_SDA: track 2.29 -> 22.5 mm
- net +3V3: track 26.3 -> 45.1 mm, vias 8 -> 30
- net Net-(U2-SC1): track 0.00 -> 18.0 mm
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- added copper zone on In2.Cu, net +3V3
- added copper zone on B.Cu, net GND
- added copper zone on In1.Cu, net GND
- removed copper zone on B.Cu, net +3V3
Other:
- board size 33.2 x 35 mm -> 60 x 50 mm
- copper layers 2 -> 4
- board text added: "LED 1"
- board text added: "LED 2"
- board text added: "Pressure MCU"
- board text added: "REV A"
- board text added: "UCM 26"
